File: switchboard1.sch (EAGLE design)
At the start: 38 parts, among them K1 S202SE2, K2 S202SE2, K3 S202SE2, K4 S202SE2, K5 S202SE2, Q1 2N7002, Q2 2N7002, Q3 2N7002, Q4 2N7002, Q5 2N7002

Commit message: nothing special...
Parts:
- R10, R11, R2, R4, R9: value 1k -> 330
- X1, X2, X3, X4, X5: value (none) -> AKL 055-02
Changed lines of the file:
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@@
 <?xml version="1.0" encoding="utf-8"?>
 <!DOCTYPE eagle SYSTEM "eagle.dtd">
-<eagle version="7.5.1">
+<eagle version="7.5.2">
 <drawing>
 <settings>
@@
 <part name="K1" library="relay" deviceset="S2*" device="" technology="02SE2"/>
 <part name="R1" library="resistor" deviceset="R-EU_" device="R0805" value="120"/>
-<part name="R2" library="resistor" deviceset="R-EU_" device="R0805" value="1k"/>
-<part name="X1" library="con-wago-508" deviceset="W237-02P" device=""/>
+<part name="R2" library="resistor" deviceset="R-EU_" device="R0805" value="330"/>
+<part name="X1" library="con-wago-508" deviceset="W237-02P" device="" value="AKL 055-02"/>
 <part name="Q1" library="adafruit" deviceset="MOSFET-N" device="REFLOW" value="2N7002"/>
 <part name="GND3" library="supply1" deviceset="GND" device=""/>
@@
 <part name="K2" library="relay" deviceset="S2*" device="" technology="02SE2"/>
 <part name="R3" library="resistor" deviceset="R-EU_" device="R0805" value="120"/>
-<part name="R4" library="resistor" deviceset="R-EU_" device="R0805" value="1k"/>
-<part name="X2" library="con-wago-508" deviceset="W237-02P" device=""/>
+<part name="R4" library="resistor" deviceset="R-EU_" device="R0805" value="330"/>
+<part name="X2" library="con-wago-508" deviceset="W237-02P" device="" value="AKL 055-02"/>
 <part name="Q2" library="adafruit" deviceset="MOSFET-N" device="REFLOW" value="2N7002"/>
 <part name="GND4" library="supply1" deviceset="GND" device=""/>
@@
 <part name="K3" library="relay" deviceset="S2*" device="" technology="02SE2"/>
 <part name="R18" library="resistor" deviceset="R-EU_" device="R0805" value="120"/>
-<part name="R9" library="resistor" deviceset="R-EU_" device="R0805" value="1k"/>
-<part name="X3" library="con-wago-508" deviceset="W237-02P" device=""/>
+<part name="R9" library="resistor" deviceset="R-EU_" device="R0805" value="330"/>
+<part name="X3" library="con-wago-508" deviceset="W237-02P" device="" value="AKL 055-02"/>
 <part name="Q3" library="adafruit" deviceset="MOSFET-N" device="REFLOW" value="2N7002"/>
 <part name="GND9" library="supply1" deviceset="GND" device=""/>
@@
 <part name="K4" library="relay" deviceset="S2*" device="" technology="02SE2"/>
 <part name="R19" library="resistor" deviceset="R-EU_" device="R0805" value="120"/>
-<part name="R10" library="resistor" deviceset="R-EU_" device="R0805" value="1k"/>
-<part name="X4" library="con-wago-508" deviceset="W237-02P" device=""/>
+<part name="R10" library="resistor" deviceset="R-EU_" device="R0805" value="330"/>
+<part name="X4" library="con-wago-508" deviceset="W237-02P" device="" value="AKL 055-02"/>
 <part name="Q4" library="adafruit" deviceset="MOSFET-N" device="REFLOW" value="2N7002"/>
 <part name="GND10" library="supply1" deviceset="GND" device=""/>
@@
 <part name="K5" library="relay" deviceset="S2*" device="" technology="02SE2"/>
 <part name="R20" library="resistor" deviceset="R-EU_" device="R0805" value="120"/>
-<part name="R11" library="resistor" deviceset="R-EU_" device="R0805" value="1k"/>
-<part name="X5" library="con-wago-508" deviceset="W237-02P" device=""/>
+<part name="R11" library="resistor" deviceset="R-EU_" device="R0805" value="330"/>
+<part name="X5" library="con-wago-508" deviceset="W237-02P" device="" value="AKL 055-02"/>
 <part name="Q5" library="adafruit" deviceset="MOSFET-N" device="REFLOW" value="2N7002"/>
 <part name="GND11" library="supply1" deviceset="GND" device=""/>
